File: Black_STM32F407VET6/STM32F407VET6.sch (KiCad schematic (older format))
At the start: 112 parts, among them J1 T0, J10 - HotBed +, J11 Heater0, J12 X_logic, J13 Microsteps, J14 X-, J15 Y-, J16 Z-, J17 Left, J18 Y_logic, J19 X+, J2 T1, J20 Y+, J21 Z+, J22 Microsteps, J23 EXP2, J24 Z_logic, J25 Bottom, J26 Microsteps, J27 EXP1, J28 E0_logic, J29 Microsteps, J3 TB, J30 Right, J31 E1_logic, J32 Microsteps, J33 X_motor, J34 Y_motor, J35 Z_motor, J36 E0_motor, J37 E1_motor, J38 X, J39 Y, J4 TC, J40 Z, J41 E0, J42 E1, J43 Heater1, J44 COM, J45 USB, J47 I2C, J48 SPI, J49 SPI, J5 + VIN -, J50 SDIO, J51 Servo, J52 Servo, J53 PowerSelect, J54 Power, J55 PD11, J56 Power, J6 Fan3, J7 Fan2, J8 Fan1, J9 Fan0, Q1 BCX70, Q10 BCX70, Q11 BCX70, Q12 IRLR8726PBF, Q13 IRLR8726PBF, Q14 IRLR8726PBF, Q2 BCX70, Q3 BCX70, Q4 IRLML0030TRPBF, Q5 BCX70, Q6 IRLML0030TRPBF, Q7 IRLML0030TRPBF, Q8 IRLML0030TRPBF, Q9 BCX70, U4 LM2596S-5, U5 AT24CS01-SSHM

Commit message: Merge of both
Parts:
- removed C11, C9: 100uF 35V, Capacitor_SMD:CP_Elec_8x6.9, symbol Device:CP_Small
- removed J12: X_logic, Connector_PinSocket_2.54mm:PinSocket_1x08_P2.54mm_Vertical, symbol STM32F407VET6:DRV_logic
- removed J13, J22, J26, J29, J32: Microsteps, Connector_PinHeader_2.54mm:PinHeader_2x03_P2.54mm_Vertical, symbol Connector_Generic:Conn_02x03_Odd_Even
- removed J14: X-, Connector_JST:JST_XH_B3B-XH-A_1x03_P2.50mm_Vertical, symbol Connector_Generic:Conn_01x03
- removed J15: Y-, Connector_JST:JST_XH_B3B-XH-A_1x03_P2.50mm_Vertical, symbol Connector_Generic:Conn_01x03
- removed J16: Z-, Connector_JST:JST_XH_B3B-XH-A_1x03_P2.50mm_Vertical, symbol Connector_Generic:Conn_01x03
- removed J17: Left, Connector_PinSocket_2.54mm:PinSocket_2x24_P2.54mm_Vertical, symbol STM32F407VET6:Left
- removed J18: Y_logic, Connector_PinSocket_2.54mm:PinSocket_1x08_P2.54mm_Vertical, symbol STM32F407VET6:DRV_logic
- removed J19: X+, Connector_JST:JST_XH_B3B-XH-A_1x03_P2.50mm_Vertical, symbol Connector_Generic:Conn_01x03
- removed J20: Y+, Connector_JST:JST_XH_B3B-XH-A_1x03_P2.50mm_Vertical, symbol Connector_Generic:Conn_01x03
- removed J21: Z+, Connector_JST:JST_XH_B3B-XH-A_1x03_P2.50mm_Vertical, symbol Connector_Generic:Conn_01x03
- removed J24: Z_logic, Connector_PinSocket_2.54mm:PinSocket_1x08_P2.54mm_Vertical, symbol STM32F407VET6:DRV_logic
- removed J25: Bottom, Connector_PinSocket_2.54mm:PinSocket_2x16_P2.54mm_Vertical, symbol STM32F407VET6:Bottom
- removed J27: EXP1, Connector_IDC:IDC-Header_2x05_P2.54mm_Vertical, symbol STM32F407VET6:EXP1
- removed J28: E0_logic, Connector_PinSocket_2.54mm:PinSocket_1x08_P2.54mm_Vertical, symbol STM32F407VET6:DRV_logic
- removed J30: Right, Connector_PinSocket_2.54mm:PinSocket_2x24_P2.54mm_Vertical, symbol STM32F407VET6:Right
- removed J31: E1_logic, Connector_PinSocket_2.54mm:PinSocket_1x08_P2.54mm_Vertical, symbol STM32F407VET6:DRV_logic
- removed J35: Z_motor, Connector_PinSocket_2.54mm:PinSocket_1x08_P2.54mm_Vertical, symbol STM32F407VET6:DRV_motor
- removed J37: E1_motor, Connector_PinSocket_2.54mm:PinSocket_1x08_P2.54mm_Vertical, symbol STM32F407VET6:DRV_motor
- removed J40: Z, Connector_JST:JST_XH_B4B-XH-A_1x04_P2.50mm_Vertical, symbol Connector_Generic:Conn_01x04
- removed J42: E1, Connector_JST:JST_XH_B4B-XH-A_1x04_P2.50mm_Vertical, symbol Connector_Generic:Conn_01x04
- removed R5, R6, R7, R8, R9: 4K7, Resistor_SMD:R_0603_1608Metric, symbol Device:R_Small
- added C?: 100uF 35V, Capacitor_SMD:CP_Elec_8x6.9, symbol Device:CP_Small
- added ESC_logic?: Conn_01x03, symbol Connector_Generic:Conn_01x03
- added J?: Right, Connector_PinSocket_2.54mm:PinSocket_2x24_P2.54mm_Vertical, symbol STM32F407VET6:Right
- added J?: Bottom, Connector_PinSocket_2.54mm:PinSocket_2x16_P2.54mm_Vertical, symbol STM32F407VET6:Bottom
- added J?: E0_logic, Connector_PinSocket_2.54mm:PinSocket_1x08_P2.54mm_Vertical, symbol STM32F407VET6-rescue:DRV_logic-STM32F407VET6
- added J?: X-, Connector_JST:JST_XH_B03B-XH-A_1x03_P2.50mm_Vertical, symbol Connector_Generic:Conn_01x03
- added J?: Z-, Connector_JST:JST_XH_B03B-XH-A_1x03_P2.50mm_Vertical, symbol Connector_Generic:Conn_01x03
- added J?: Y-, Connector_JST:JST_XH_B03B-XH-A_1x03_P2.50mm_Vertical, symbol Connector_Generic:Conn_01x03
- added J?: Z+, Connector_JST:JST_XH_B03B-XH-A_1x03_P2.50mm_Vertical, symbol Connector_Generic:Conn_01x03
- added J?: X_logic, Connector_PinSocket_2.54mm:PinSocket_1x08_P2.54mm_Vertical, symbol STM32F407VET6-rescue:DRV_logic-STM32F407VET6
- added J?: Y_logic, Connector_PinSocket_2.54mm:PinSocket_1x08_P2.54mm_Vertical, symbol STM32F407VET6-rescue:DRV_logic-STM32F407VET6
- added J?: Z_logic, Connector_PinSocket_2.54mm:PinSocket_1x08_P2.54mm_Vertical, symbol STM32F407VET6-rescue:DRV_logic-STM32F407VET6
- added J?: Z_motor, Connector_PinSocket_2.54mm:PinSocket_1x08_P2.54mm_Vertical, symbol STM32F407VET6:DRV_motor
- added J?: Left, Connector_PinSocket_2.54mm:PinSocket_2x24_P2.54mm_Vertical, symbol STM32F407VET6:Left
- added J? (x2): Z, Connector_JST:JST_XH_B04B-XH-A_1x04_P2.50mm_Vertical, symbol Connector_Generic:Conn_01x04
- added J?: LCD2004, symbol STM32F407VET6:LCD2004
- added J?: LIGHTS, symbol Connector_Generic:Conn_01x03
- added J?: UNUSED_PINS, symbol Connector_Generic:Conn_01x05
- added JXXX?: ESC_POWER, TerminalBlock_MetzConnect:TerminalBlock_MetzConnect_Type055_RT01502HDWU_1x02_P5.00mm_Horizontal, symbol Connector:Screw_Terminal_01x02
Connections:
- net labels added: E0_CS, KEYPAD_PIN, LIGHT_DIN, PA15, PB8, PE1, PE3, PE4, SPINDLE_PIN, Tmc_MISO, Tmc_MOSI, Tmc_SCK, X_CS, Y_CS, Z_CS
- net labels removed: E1_Dir, E1_En, E1_Step, X+, Y+
- wire segments 243 -> 212
- no-connect marks 27 -> 32
Other:
- moved on the sheet: C10, J36, J41, J49

Commit message: Arranged parts on PCB, swapped a few pins in schematic to align connectors.
Parts:
- removed C5: 100uF 35V, Capacitor_THT:CP_Radial_D8.0mm_P3.50mm, symbol Device:CP_Small
- removed C6: 220uF 35V, Capacitor_THT:CP_Radial_D6.3mm_P2.50mm, symbol Device:CP_Small
- removed D1: SS14, Diode_SMD:D_SMA, symbol Diode:B120-E3
- removed ESC_logic?: Conn_01x03, symbol Connector_Generic:Conn_01x03
- removed J45: USB, Connector_PinHeader_2.54mm:PinHeader_1x04_P2.54mm_Vertical, symbol Connector_Generic:Conn_01x04
- removed J?: UNUSED_PINS, symbol Connector_Generic:Conn_01x05
- removed L1: 47uH, Inductor_THT:L_Radial_D9.5mm_P5.00mm_Fastron_07HVP, symbol Device:L_Small
- removed U4: LM2596S-5, Package_TO_SOT_SMD:TO-263-5_TabPin3, symbol Regulator_Switching:LM2596S-5
- added J16: USB_B, Connector_USB:USB_B_OST_USB-B1HSxx_Horizontal, symbol Connector:USB_B
- added R5: 1,5k, Resistor_SMD:R_0603_1608Metric, symbol Device:R_Small
- J12, J13, J14, J15: renamed from J?; footprint Connector_JST:JST_XH_B03B-XH-A_1x03_P2.50mm_Vertical -> Connector_JST:JST_XH_B3B-XH-A_1x03_P2.50mm_Vertical
- J24: renamed from J?; footprint (none) -> Connector_JST:JST_XH_B10B-XH-A_1x10_P2.50mm_Vertical
- J28: renamed from J?; footprint (none) -> Connector_JST:JST_XH_B3B-XH-A_1x03_P2.50mm_Vertical
- J29, J30: renamed from J?; footprint Connector_JST:JST_XH_B04B-XH-A_1x04_P2.50mm_Vertical -> Connector_JST:JST_XH_B4B-XH-A_1x04_P2.50mm_Vertical
- gave numbers to parts that had none: 10
Connections:
- net labels removed: PA15, PB8, PE1, PE3, PE4, SPINDLE_PIN
- wire segments 212 -> 209
- no-connect marks 32 -> 31
Other:
- note removed: "Já nevím, jak je to tady myšlený, ale 5v co jde z USB by nemělo být spojené s výstupem z toho 5v spínaného měniče. Těch 5v z USB pravděpodobně vůbec není potřeba zapojovat. 5v v sekci e8, potenciálně konektor j56, jestli to je vstup.\n"
- moved on the sheet: J10, J11, J12, J13, J14, J15, J22, J26, J43, J44, J47, J48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

Commit message: Flash button, Endstops, Drivers moved
Parts:
- added R6: R4.7K, Resistor_SMD:R_0603_1608Metric, symbol Device:R
- added SW1: Boot0, Button_Switch_THT:SW_PUSH_6mm_H5mm, symbol Switch:SW_Push
Connections:
- net +3V3: now also SW1.1
- net GND: now also R6.1; no longer J26.5 (BOOT0)
- net LCD4: now also J25.15 (PD1); no longer J25.5 (PD8)
- net LCD5: now also J25.11 (PE10); no longer J25.9 (PE12)
- net LCD6: now also J25.7 (PE14); no longer J25.13 (PE8)
- net LCD7: now also J25.5 (PD8); no longer J25.15 (PD1)
- net LCDE: now also J25.9 (PE12); no longer J25.11 (PE10)
- net LCDRS: now also J25.13 (PE8); no longer J25.7 (PE14)
- net X-: now also J25.14 (PE7); no longer J22.16 (PC13)
- net X_Dir: now also J22.31 (PC4); no longer J26.20 (PD6)
- net X_En: now also J22.15 (PE6); no longer J22.35 (PE7)
- net X_Step: now also J22.11 (PE2); no longer J22.31 (PC4)
- net Y_Dir: now also J22.16 (PC13); no longer J22.11 (PE2)
- net Y_En: now also J26.20 (PD6); no longer J22.15 (PE6)
- new net: J26.5 (BOOT0), R6.2, SW1.2
Changed lines of the file:
@@
-$EndComp
-$Comp
-L STM32F407VET6:Right J26
-U 1 1 5D30CC8F
-P 10900 2750
-F 0 "J26" H 10900 4165 50  0000 C CNN
-F 1 "Right" H 10900 4074 50  0000 C CNN
-F 2 "Connector_PinSocket_2.54mm:PinSocket_2x24_P2.54mm_Vertical" H 10900 2400 50  0001 C CNN
-F 3 "" H 10900 2400 50  0001 C CNN
-	1    10900 2750
-	1    0    0    -1
 $EndComp
 $Comp
@@
 Text GLabel 10550 1600 0    50   Input ~ 0
 3V3
-Text GLabel 10550 1700 0    50   Input ~ 0
-3V3
 Text GLabel 8850 1750 2    50   Input ~ 0
 3V3
@@
 3V3
 Text GLabel 8150 1950 0    50   Input ~ 0
-GND
-Text GLabel 10550 1900 0    50   Input ~ 0
 GND
 Text GLabel 10550 2000 0    50   Input ~ 0
@@
 Text GLabel 8150 1650 0    50   Input ~ 0
 5V
-Wire Wire Line
-	10550 1900 10550 1800
 Text GLabel 9500 8500 3    50   Input ~ 0
 5V
@@
 Text GLabel 10300 5850 3    50   Input ~ 0
 ENC
+Text GLabel 9800 5150 1    50   Input ~ 0
+LCDRS
+Text GLabel 10000 5150 1    50   Input ~ 0
+LCDE
+Text GLabel 9700 5150 1    50   Input ~ 0
+LCD4
+Text GLabel 9900 5150 1    50   Input ~ 0
+LCD5
 Text GLabel 10100 5150 1    50   Input ~ 0
-LCDRS
-Text GLabel 9900 5150 1    50   Input ~ 0
-LCDE
+LCD6
 Text GLabel 10200 5150 1    50   Input ~ 0
-LCD4
-Text GLabel 10000 5150 1    50   Input ~ 0
-LCD5
-Text GLabel 9800 5150 1    50   Input ~ 0
-LCD6
-Text GLabel 9700 5150 1    50   Input ~ 0
 LCD7
 Text GLabel 4400 9450 3    50   Input ~ 0
@@
 NoConn ~ 8850 3350
 NoConn ~ 8850 3250
-Text GLabel 8150 2050 0    50   Input ~ 0
+Text GLabel 8850 2250 2    50   Input ~ 0
 Y_Dir
-Text GLabel 8150 2250 0    50   Input ~ 0
+Text GLabel 11250 2500 2    50   Input ~ 0
 Y_En
 Text GLabel 8850 2150 2    50   Input ~ 0
 Y_Step
-Text GLabel 8850 2250 2    50   Input ~ 0
+Text GLabel 9800 5850 3    50   Input ~ 0
 X-
 Text GLabel 8850 2650 2    50   Input ~ 0
@@
 Text GLabel 8150 2750 0    50   Input ~ 0
 Heater0
-Text GLabel 11250 2500 2    50   Input ~ 0
+Text GLabel 8150 3050 0    50   Input ~ 0
 X_Dir
 Text GLabel 8850 2750 2    50   Input ~ 0
@@
 Y-
 NoConn ~ 8850 3050
-Text GLabel 8150 3050 0    50   Input ~ 0
+Text GLabel 8150 2050 0    50   Input ~ 0
 X_Step
 NoConn ~ 8850 3150
-Text GLabel 8150 3250 0    50   Input ~ 0
+Text GLabel 8150 2250 0    50   Input ~ 0
 X_En
 Text GLabel 8150 3750 0    50   Input ~ 0
@@
 NoConn ~ 9600 5850
 NoConn ~ 9700 5850
-NoConn ~ 9800 5850
 NoConn ~ 9600 5150
 NoConn ~ 10550 2800
@@
 	1    0    0    -1
 $EndComp
+NoConn ~ 8150 3250
+$Comp
+L STM32F407VET6:Right J26
+U 1 1 5D30CC8F
+P 10900 2750
+F 0 "J26" H 10900 4165 50  0000 C CNN
+F 1 "Right" H 10900 4074 50  0000 C CNN
+F 2 "Connector_PinSocket_2.54mm:PinSocket_2x24_P2.54mm_Vertical" H 10900 2400 50  0001 C CNN
+F 3 "" H 10900 2400 50  0001 C CNN
+	1    10900 2750
+	1    0    0    -1
+$EndComp
+Text GLabel 10550 1900 0    50   Input ~ 0
+GND
+Text GLabel 10550 1700 0    50   Input ~ 0
+3V3
+$Comp
+L Switch:SW_Push SW1
+U 1 1 5D48E2E2
+P 10050 1950
+F 0 "SW1" V 10096 1902 50  0000 R CNN
+F 1 "Boot0" V 10005 1902 50  0000 R CNN
+F 2 "Button_Switch_THT:SW_PUSH_6mm_H5mm" H 10050 2150 50  0001 C CNN
+F 3 "~" H 10050 2150 50  0001 C CNN
+	1    10050 1950
+	0    -1   -1   0
+$EndComp
+$Comp
+L Device:R R6
+U 1 1 5D4F03A2
+P 10050 1600
+F 0 "R6" H 10120 1646 50  0000 L CNN
+F 1 "R4.7K" H 10120 1555 50  0000 L CNN
+F 2 "Resistor_SMD:R_0603_1608Metric" V 9980 1600 50  0001 C CNN
+F 3 "~" H 10050 1600 50  0001 C CNN
+	1    10050 1600
+	1    0    0    -1
+$EndComp
+Text GLabel 10050 1450 1    50   Input ~ 0
+GND
+Text GLabel 10050 2150 3    50   Input ~ 0
+3V3
+Wire Wire Line
+	10050 1800 10550 1800
+Wire Wire Line
+	10050 1750 10050 1800
+Connection ~ 10050 1750
 $EndSCHEMATC
